File: pcb/ModusBatteryMonitor.kicad_pcb (KiCad board)
At the start: 2 copper layers, 70.6 x 28 mm, 17 parts, among them IC101 ATTINY3224-SS, IC102 MAX485/3485, P101 RS485, P102 NTC1, P103 NTC2, P104 DEBUG, P105 SHUNT+, P106 SHUNT-, P107 BAT-, U101 NCP1117ST50T3G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

Commit message: Made housing
Connections:
- IC102 pad 6: RS485-B -> RS485-A
- IC102 pad 7: RS485-A -> RS485-B
Routing:
- net RS485-A: track 14.0 -> 22.9 mm, vias 1 -> 2
- net RS485-B: track 19.1 -> 10.1 mm, vias 1 -> 0
Other:
- net class Default: trace_width 1 -> 0.8
Changed lines of the file:
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@@
   (general
     (links 41)
-    (no_connects 0)
-    (area 102.755559 65.600909 209.700001 120.600128)
+    (no_connects 2)
+    (area 119.624999 74.024999 190.375001 102.175001)
     (thickness 1.6)
     (drawings 45)
@@
   )
   (setup
-    (last_trace_width 1)
+    (last_trace_width 0.8)
     (trace_clearance 0.2)
     (zone_clearance 0.5)
@@
   (net_class Default "This is the default net class."
     (clearance 0.2)
-    (trace_width 1)
+    (trace_width 0.8)
     (via_dia 2)
     (via_drill 0.7)
@@
       (net 2 GND))
     (pad 6 smd rect (at 2.7 0.635) (size 1.55 0.6) (layers F.Cu F.Paste F.Mask)
+      (net 16 RS485-A))
+    (pad 7 smd rect (at 2.7 -0.635) (size 1.55 0.6) (layers F.Cu F.Paste F.Mask)
       (net 18 RS485-B))
-    (pad 7 smd rect (at 2.7 -0.635) (size 1.55 0.6) (layers F.Cu F.Paste F.Mask)
-      (net 16 RS485-A))
     (pad 8 smd rect (at 2.7 -1.905) (size 1.55 0.6) (layers F.Cu F.Paste F.Mask)
       (net 3 5V))
@@
   (gr_line (start 190.3 74.1) (end 190.3 102.1) (angle 90) (layer Edge.Cuts) (width 0.15))
   (gr_line (start 120.4 74.1) (end 190.3 74.1) (angle 90) (layer Edge.Cuts) (width 0.15))
-  (segment (start 172.2 86.85) (end 173.5 86.85) (width 1) (layer F.Cu) (net 1) (status 400000))
-  (segment (start 173.15 91.33) (end 174.13 92.31) (width 1) (layer B.Cu) (net 1) (status 800000))
+  (segment (start 172.2 86.85) (end 173.5 86.85) (width 1) (layer F.Cu) (net 1))
+  (segment (start 173.15 91.33) (end 174.13 92.31) (width 1) (layer B.Cu) (net 1))
   (segment (start 173.15 87.3) (end 173.15 91.33) (width 1) (layer B.Cu) (net 1))
   (segment (start 173.55 86.9) (end 173.15 87.3) (width 1) (layer B.Cu) (net 1))
@@
   (segment (start 166.15 86.85) (end 161.65 86.85) (width 1) (layer B.Cu) (net 2))
   (segment (start 161.65 86.85) (end 160.7 85.9) (width 1) (layer B.Cu) (net 2))
-  (segment (start 167.3 84.05) (end 167.3 86.05) (width 1) (layer F.Cu) (net 2) (status 400000))
+  (segment (start 167.3 84.05) (end 167.3 86.05) (width 1) (layer F.Cu) (net 2))
   (segment (start 167.3 86.05) (end 168.1 86.85) (width 1) (layer F.Cu) (net 2))
-  (segment (start 169.05 89.77) (end 166.68 89.77) (width 1) (layer B.Cu) (net 2) (status 400000))
+  (segment (start 169.05 89.77) (end 166.68 89.77) (width 1) (layer B.Cu) (net 2))
   (segment (start 166.68 89.77) (end 166.15 89.24) (width 1) (layer B.Cu) (net 2))
   (segment (start 166.15 89.24) (end 166.15 86.85) (width 1) (layer B.Cu) (net 2))
   (via (at 166.15 86.85) (size 2) (drill 0.7) (layers F.Cu B.Cu) (net 2))
   (segment (start 166.15 86.85) (end 168.1 86.85) (width 1) (layer F.Cu) (net 2))
-  (segment (start 168.1 86.85) (end 169.2 86.85) (width 1) (layer F.Cu) (net 2) (status 800000))
+  (segment (start 168.1 86.85) (end 169.2 86.85) (width 1) (layer F.Cu) (net 2))
   (segment (start 159.4 96.2) (end 159.4 96.15) (width 0.5) (layer F.Cu) (net 2))
-  (segment (start 157.85 94.6) (end 157.85 91.955) (width 0.5) (layer F.Cu) (net 2) (status 800000))
+  (segment (start 157.85 94.6) (end 157.85 91.955) (width 0.5) (layer F.Cu) (net 2))
   (segment (start 159.4 96.15) (end 157.85 94.6) (width 0.5) (layer F.Cu) (net 2))
   (segment (start 169.05 99.93) (end 163.13 99.93) (width 1) (layer B.Cu) (net 2))
@@
   (segment (start 142.6 91.81) (end 136.35 91.81) (width 0.5) (layer F.Cu) (net 2))
   (segment (start 136.35 91.81) (end 135.8 92.36) (width 0.5) (layer F.Cu) (net 2))
-  (segment (start 157.85 88.145) (end 156.455 88.145) (width 0.5) (layer F.Cu) (net 3) (status 400000))
-  (segment (start 155.95 94) (end 154.75 94) (width 0.5) (layer F.Cu) (net 3) (status 800000))
+  (segment (start 157.85 88.145) (end 156.455 88.145) (width 0.5) (layer F.Cu) (net 3))
+  (segment (start 155.95 94) (end 154.75 94) (width 0.5) (layer F.Cu) (net 3))
   (segment (start 156.05 93.9) (end 155.95 94) (width 0.5) (layer F.Cu) (net 3))
   (segment (start 156.05 88.55) (end 156.05 93.9) (width 0.5) (layer F.Cu) (net 3))
   (segment (start 156.455 88.145) (end 156.05 88.55) (width 0.5) (layer F.Cu) (net 3))
-  (segment (start 157.9 88.095) (end 157.9 86.795) (width 0.5) (layer F.Cu) (net 3) (status 400000))
+  (segment (start 157.9 88.095) (end 157.9 86.795) (width 0.5) (layer F.Cu) (net 3))
   (segment (start 157.9 82.35) (end 158.15 82.1) (width 0.5) (layer F.Cu) (net 3))
   (segment (start 157.9 86.795) (end 157.9 82.35) (width 1) (layer F.Cu) (net 3))
-  (segment (start 157.9 88.095) (end 157.85 88.145) (width 0.5) (layer F.Cu) (net 3) (status C00000))
+  (segment (start 157.9 88.095) (end 157.85 88.145) (width 0.5) (layer F.Cu) (net 3))
   (segment (start 164.5 82.3) (end 164.5 78.35) (width 1) (layer F.Cu) (net 3))
   (segment (start 164.5 78.35) (end 165.1 77.75) (width 1) (layer F.Cu) (net 3))
@@
   (segment (start 147.75 94.65) (end 147.75 93.55) (width 0.5) (layer F.Cu) (net 3))
   (segment (start 147.5 94.9) (end 147.75 94.65) (width 0.5) (layer F.Cu) (net 3))
-  (segment (start 152.45 90.685) (end 152.45 89.415) (width 0.5) (layer F.Cu) (net 4) (status C00000))
-  (segment (start 148 90.54) (end 149.19 90.54) (width 0.5) (layer F.Cu) (net 4) (status 400000))
-  (segment (start 149.5 90.85) (end 152.285 90.85) (width 0.5) (layer F.Cu) (net 4) (status 800000))
+  (segment (start 152.45 90.685) (end 152.45 89.415) (width 0.5) (layer F.Cu) (net 4))
+  (segment (start 148 90.54) (end 149.19 90.54) (width 0.5) (layer F.Cu) (net 4))
+  (segment (start 149.5 90.85) (end 152.285 90.85) (width 0.5) (layer F.Cu) (net 4))
   (segment (start 149.19 90.54) (end 149.5 90.85) (width 0.5) (layer F.Cu) (net 4))
-  (segment (start 152.285 90.85) (end 152.45 90.685) (width 0.5) (layer F.Cu) (net 4) (status C00000))
+  (segment (start 152.285 90.85) (end 152.45 90.685) (width 0.5) (layer F.Cu) (net 4))
   (segment (start 148 89.27) (end 150.17 89.27) (width 0.5) (layer F.Cu) (net 5))
   (segment (start 150.4 89.5) (end 150.4 97.95) (width 0.5) (layer B.Cu) (net 5))
@@
   (segment (start 154.8 97.95) (end 154.8 95.95) (width 0.5) (layer F.Cu) (net 6))
   (segment (start 154.8 95.95) (end 154.75 95.9) (width 0.5) (layer F.Cu) (net 6))
-  (segment (start 148 85.46) (end 152.24 85.46) (width 0.5) (layer F.Cu) (net 7) (status 400000))
-  (segment (start 152.45 85.67) (end 152.45 88.145) (width 0.5) (layer F.Cu) (net 7) (status 800000))
+  (segment (start 148 85.46) (end 152.24 85.46) (width 0.5) (layer F.Cu) (net 7))
+  (segment (start 152.45 85.67) (end 152.45 88.145) (width 0.5) (layer F.Cu) (net 7))
   (segment (start 152.24 85.46) (end 152.45 85.67) (width 0.5) (layer F.Cu) (net 7))
-  (segment (start 148 84.19) (end 153.54 84.19) (width 0.5) (layer F.Cu) (net 8) (status 400000))
-  (segment (start 153.745 91.955) (end 152.45 91.955) (width 0.5) (layer F.Cu) (net 8) (status 800000))
+  (segment (start 148 84.19) (end 153.54 84.19) (width 0.5) (layer F.Cu) (net 8))
+  (segment (start 153.745 91.955) (end 152.45 91.955) (width 0.5) (layer F.Cu) (net 8))
   (segment (start 154.45 91.25) (end 153.745 91.955) (width 0.5) (layer F.Cu) (net 8))
   (segment (start 154.45 85.1) (end 154.45 91.25) (width 0.5) (layer F.Cu) (net 8))
@@
   (segment (start 178 74.7) (end 181.5 78.2) (width 1) (layer F.Cu) (net 15))
   (segment (start 147.09 77.98) (end 147.09 76.76) (width 1) (layer F.Cu) (net 15))
-  (segment (start 157.85 89.415) (end 160.385 89.415) (width 0.5) (layer F.Cu) (net 16) (status 400000))
-  (segment (start 167.05 94.85) (end 169.05 94.85) (width 0.5) (layer B.Cu) (net 16) (status 800000))
   (segment (start 161 88.8) (end 167.05 94.85) (width 0.5) (layer B.Cu) (net 16))
+  (segment (start 167.05 94.85) (end 169.05 94.85) (width 0.5) (layer B.Cu) (net 16))
+  (segment (start 157.85 90.685) (end 159.885 90.685) (width 0.5) (layer F.Cu) (net 16))
+  (segment (start 159.885 90.685) (end 160.85 91.65) (width 0.5) (layer F.Cu) (net 16))
+  (via (at 160.85 91.65) (size 2) (drill 0.7) (layers F.Cu B.Cu) (net 16))
+  (segment (start 160.85 91.65) (end 166.59 97.39) (width 0.5) (layer B.Cu) (net 16))
   (via (at 161 88.8) (size 2) (drill 0.7) (layers F.Cu B.Cu) (net 16))
   (segment (start 160.385 89.415) (end 161 88.8) (width 0.5) (layer F.Cu) (net 16))
   (segment (start 139.4 84.25) (end 136.29 84.25) (width 0.5) (layer F.Cu) (net 17))
   (segment (start 136.29 84.25) (end 135.8 84.74) (width 0.5) (layer F.Cu) (net 17))
-  (segment (start 157.85 90.685) (end 159.885 90.685) (width 0.5) (layer F.Cu) (net 18) (status 400000))
-  (segment (start 166.59 97.39) (end 174.13 97.39) (width 0.5) (layer B.Cu) (net 18) (status 800000))
-  (segment (start 160.85 91.65) (end 166.59 97.39) (width 0.5) (layer B.Cu) (net 18))
-  (via (at 160.85 91.65) (size 2) (drill 0.7) (layers F.Cu B.Cu) (net 18))
-  (segment (start 159.885 90.685) (end 160.85 91.65) (width 0.5) (layer F.Cu) (net 18))
+  (segment (start 157.85 89.415) (end 160.385 89.415) (width 0.5) (layer F.Cu) (net 18))
+  (segment (start 166.59 97.39) (end 174.13 97.39) (width 0.5) (layer B.Cu) (net 18))
   (zone (net 0) (net_name "") (layer B.Cu) (hatch edge 0.508)
     (connect_pads (clearance 0.5))
@@
     (connect_pads (clearance 0.5))
     (min_thickness 1)
-    (fill yes (arc_segments 16) (thermal_gap 0.508) (thermal_bridge_width 1.1) (smoothing fillet))
+    (fill (arc_segments 16) (thermal_gap 0.508) (thermal_bridge_width 1.1) (smoothing fillet))
     (polygon
       (pts
@@
     (connect_pads (clearance 0.5))
     (min_thickness 1)
-    (fill yes (arc_segments 16) (thermal_gap 0.508) (thermal_bridge_width 1.1) (smoothing fillet))
+    (fill (arc_segments 16) (thermal_gap 0.508) (thermal_bridge_width 1.1) (smoothing fillet))
     (polygon
       (pts

Commit message: Fixed NtC sensors and adjusted LUT
Connections:
- P101 pad 3: RS485-A -> RS485-B
- P101 pad 4: RS485-B -> RS485-A
Routing:
- net RS485-A: track 22.9 -> 19.1 mm, vias 2 -> 1
- net RS485-B: track 10.1 -> 14.0 mm, vias 0 -> 1
Changed lines of the file:
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@@
   (general
     (links 41)
-    (no_connects 2)
+    (no_connects 0)
     (area 119.624999 74.024999 190.375001 102.175001)
     (thickness 1.6)
@@
     (fp_line (start -6.35 -7.62) (end -6.35 3.81) (layer F.SilkS) (width 0.15))
     (pad 3 thru_hole circle (at 0 0 270) (size 2 2) (drill 0.762) (layers *.Cu *.Mask)
-      (net 16 RS485-A))
+      (net 18 RS485-B))
     (pad 2 thru_hole circle (at -2.54 -5.08 270) (size 2 2) (drill 0.762) (layers *.Cu *.Mask)
       (net 1 VIn))
@@
       (net 2 GND))
     (pad 4 thru_hole circle (at 2.54 -5.08 270) (size 2 2) (drill 0.762) (layers *.Cu *.Mask)
-      (net 18 RS485-B))
+      (net 16 RS485-A))
     (pad 5 thru_hole circle (at 5.08 0 270) (size 2 2) (drill 0.762) (layers *.Cu *.Mask)
       (net 2 GND))
@@
   (segment (start 178 74.7) (end 181.5 78.2) (width 1) (layer F.Cu) (net 15))
   (segment (start 147.09 77.98) (end 147.09 76.76) (width 1) (layer F.Cu) (net 15))
-  (segment (start 161 88.8) (end 167.05 94.85) (width 0.5) (layer B.Cu) (net 16))
-  (segment (start 167.05 94.85) (end 169.05 94.85) (width 0.5) (layer B.Cu) (net 16))
   (segment (start 157.85 90.685) (end 159.885 90.685) (width 0.5) (layer F.Cu) (net 16))
   (segment (start 159.885 90.685) (end 160.85 91.65) (width 0.5) (layer F.Cu) (net 16))
   (via (at 160.85 91.65) (size 2) (drill 0.7) (layers F.Cu B.Cu) (net 16))
   (segment (start 160.85 91.65) (end 166.59 97.39) (width 0.5) (layer B.Cu) (net 16))
-  (via (at 161 88.8) (size 2) (drill 0.7) (layers F.Cu B.Cu) (net 16))
-  (segment (start 160.385 89.415) (end 161 88.8) (width 0.5) (layer F.Cu) (net 16))
+  (segment (start 166.59 97.39) (end 174.13 97.39) (width 0.5) (layer B.Cu) (net 16))
   (segment (start 139.4 84.25) (end 136.29 84.25) (width 0.5) (layer F.Cu) (net 17))
   (segment (start 136.29 84.25) (end 135.8 84.74) (width 0.5) (layer F.Cu) (net 17))
+  (segment (start 161 88.8) (end 167.05 94.85) (width 0.5) (layer B.Cu) (net 18))
+  (segment (start 167.05 94.85) (end 169.05 94.85) (width 0.5) (layer B.Cu) (net 18))
+  (via (at 161 88.8) (size 2) (drill 0.7) (layers F.Cu B.Cu) (net 18))
+  (segment (start 160.385 89.415) (end 161 88.8) (width 0.5) (layer F.Cu) (net 18))
   (segment (start 157.85 89.415) (end 160.385 89.415) (width 0.5) (layer F.Cu) (net 18))
-  (segment (start 166.59 97.39) (end 174.13 97.39) (width 0.5) (layer B.Cu) (net 18))
   (zone (net 0) (net_name "") (layer B.Cu) (hatch edge 0.508)
     (connect_pads (clearance 0.5))
